File: designs/weather_stations/qwels weather station/PCB/weather.kicad_pcb (KiCad board)
At the start: 2 copper layers, 58 x 34.5 mm, 4 parts, among them U1 WEMOS_C3_Mini, U2 TFT_ST7735_SD, U3 AM2302

Commit message: Updated
Connections:
- U1 pad 11: Net-(U1-SCK/IO6) -> SCK
- U1 pad 12: Net-(U1-MOSI/IO7) -> MOSI
- U1 pad 2: unconnected-(U1-IO3-Pad2) -> cs
- U1 pad 3: unconnected-(U1-MISO/IO2-Pad3) -> MISO
- U1 pad 4: unconnected-(U1-IO1-Pad4) -> Net-(U1-IO1)
- U1 pad 5: unconnected-(U1-IO0-Pad5) -> Net-(U1-IO0)
- U2 pad 10: unconnected-(U2-SD_MOSI-Pad10) -> MOSI
- U2 pad 11: unconnected-(U2-SD_MISO-Pad11) -> MISO
- U2 pad 12: unconnected-(U2-SD_SCK-Pad12) -> SCK
- U2 pad 6: Net-(U1-MOSI/IO7) -> Net-(U1-IO0)
- U2 pad 7: Net-(U1-SCK/IO6) -> Net-(U1-IO1)
- U2 pad 9: unconnected-(U2-SD_CS-Pad9) -> cs
Routing:
- net SCK: track 0.00 -> 61.6 mm, vias 0 -> 1
- net MOSI: track 0.00 -> 52.1 mm, vias 0 -> 1
- net MISO: track 0.00 -> 44.0 mm
- net cs: track 0.00 -> 42.2 mm
- net Net-(U1-SCK/IO6): track 29.1 -> 0.00 mm
- net Net-(U1-MOSI/IO7): track 24.9 -> 0.00 mm, vias 2 -> 0
- net Net-(U1-IO0): track 0.00 -> 24.0 mm
- net Net-(U1-IO1): track 0.00 -> 19.5 mm
- net SDA: track 62.6 -> 66.6 mm
- net Net-(U2-LED): track 60.8 -> 61.0 mm, vias 0 -> 1
