File: designs/weather_stations/qwels weather station/PCB/weather.kicad_sch (KiCad schematic)
At the start: 4 parts, among them U1 WEMOS_C3_Mini, U2 TFT_ST7735_SD, U3 AM2302

Commit message: Updated
Connections:
- net MOSI: now reaches U2.10 (SD_MOSI)
- net MOSI: now also U1.12 (MOSI/IO7)
- net MISO: now reaches U2.11 (SD_MISO)
- net MISO: now also U1.3 (MISO/IO2)
- net SCK: now reaches U2.12 (SD_SCK)
- net SCK: now also U1.11 (SCK/IO6)
- net at U2.6 (LCD_MOSI): now also U1.5 (IO0); no longer U1.12 (MOSI/IO7)
- net at U2.7 (LCD_SCK): now also U1.4 (IO1); no longer U1.11 (SCK/IO6)
- net cs: now reaches U2.9 (SD_CS)
- net cs: now also U1.2 (IO3)
Changed lines of the file:
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@@
 	(wire
 		(pts
-			(xy 129.54 86.36) (xy 129.54 88.9)
+			(xy 127 91.44) (xy 135.89 91.44)
 		)
 		(stroke
@@
 	(wire
 		(pts
-			(xy 133.35 83.82) (xy 127 83.82)
-		)
-		(stroke
-			(width 0)
-			(type default)
-		)
-	)
-	(wire
-		(pts
 			(xy 137.16 73.66) (xy 137.16 91.44)
 		)
@@
 	(wire
 		(pts
-			(xy 146.05 86.36) (xy 133.35 86.36)
+			(xy 135.89 86.36) (xy 146.05 86.36)
 		)
 		(stroke
@@
 	(wire
 		(pts
-			(xy 129.54 88.9) (xy 146.05 88.9)
-		)
-		(stroke
-			(width 0)
-			(type default)
-		)
-	)
-	(wire
-		(pts
-			(xy 133.35 86.36) (xy 133.35 83.82)
-		)
-		(stroke
-			(width 0)
-			(type default)
-		)
-	)
-	(wire
-		(pts
 			(xy 127 78.74) (xy 146.05 78.74)
 		)
@@
 	(wire
 		(pts
+			(xy 135.89 91.44) (xy 135.89 86.36)
+		)
+		(stroke
+			(width 0)
+			(type default)
+		)
+	)
+	(wire
+		(pts
 			(xy 137.16 91.44) (xy 146.05 91.44)
 		)
@@
 	(wire
 		(pts
-			(xy 127 86.36) (xy 129.54 86.36)
+			(xy 127 88.9) (xy 146.05 88.9)
 		)
 		(stroke
@@
 		)
 	)
+	(global_label "MISO"
+		(shape input)
+		(at 170.18 86.36 0)
+		(fields_autoplaced yes)
+		(effects
+			(font
+				(size 1.27 1.27)
+			)
+			(justify left)
+		)
+		(property "Intersheetrefs" "${INTERSHEET_REFS}"
+			(at 177.7614 86.36 0)
+			(effects
+				(font
+					(size 1.27 1.27)
+				)
+				(justify left)
+				(hide yes)
+			)
+		)
+	)
 	(global_label "3v"
 		(shape input)
@@
 		)
 	)
+	(global_label "MISO"
+		(shape input)
+		(at 127 76.2 0)
+		(fields_autoplaced yes)
+		(effects
+			(font
+				(size 1.27 1.27)
+			)
+			(justify left)
+		)
+		(property "Intersheetrefs" "${INTERSHEET_REFS}"
+			(at 134.5814 76.2 0)
+			(effects
+				(font
+					(size 1.27 1.27)
+				)
+				(justify left)
+				(hide yes)
+			)
+		)
+	)
 	(global_label "gnd"
 		(shape input)
@@
 		)
 	)
+	(global_label "MOSI"
+		(shape input)
+		(at 127 83.82 0)
+		(fields_autoplaced yes)
+		(effects
+			(font
+				(size 1.27 1.27)
+			)
+			(justify left)
+		)
+		(property "Intersheetrefs" "${INTERSHEET_REFS}"
+			(at 134.5814 83.82 0)
+			(effects
+				(font
+					(size 1.27 1.27)
+				)
+				(justify left)
+				(hide yes)
+			)
+		)
+	)
 	(global_label "gnd"
 		(shape input)
@@
 		)
 	)
+	(global_label "cs"
+		(shape input)
+		(at 127 73.66 0)
+		(fields_autoplaced yes)
+		(effects
+			(font
+				(size 1.27 1.27)
+			)
+			(justify left)
+		)
+		(property "Intersheetrefs" "${INTERSHEET_REFS}"
+			(at 132.1019 73.66 0)
+			(effects
+				(font
+					(size 1.27 1.27)
+				)
+				(justify left)
+				(hide yes)
+			)
+		)
+	)
 	(global_label "gnd"
 		(shape input)
@@
 		)
 	)
+	(global_label "cs"
+		(shape input)
+		(at 170.18 81.28 0)
+		(fields_autoplaced yes)
+		(effects
+			(font
+				(size 1.27 1.27)
+			)
+			(justify left)
+		)
+		(property "Intersheetrefs" "${INTERSHEET_REFS}"
+			(at 175.2819 81.28 0)
+			(effects
+				(font
+					(size 1.27 1.27)
+				)
+				(justify left)
+				(hide yes)
+			)
+		)
+	)
+	(global_label "SCK"
+		(shape input)
+		(at 170.18 88.9 0)
+		(fields_autoplaced yes)
+		(effects
+			(font
+				(size 1.27 1.27)
+			)
+			(justify left)
+		)
+		(property "Intersheetrefs" "${INTERSHEET_REFS}"
+			(at 176.9147 88.9 0)
+			(effects
+				(font
+					(size 1.27 1.27)
+				)
+				(justify left)
+				(hide yes)
+			)
+		)
+	)
 	(global_label "SDA"
 		(shape input)
@@
 		)
 	)
+	(global_label "MOSI"
+		(shape input)
+		(at 170.18 83.82 0)
+		(fields_autoplaced yes)
+		(effects
+			(font
+				(size 1.27 1.27)
+			)
+			(justify left)
+		)
+		(property "Intersheetrefs" "${INTERSHEET_REFS}"
+			(at 177.7614 83.82 0)
+			(effects
+				(font
+					(size 1.27 1.27)
+				)
+				(justify left)
+				(hide yes)
+			)
+		)
+	)
 	(global_label "3v"
 		(shape input)
@@
 			(effects
 				(font
+					(size 1.27 1.27)
+				)
+				(justify left)
+				(hide yes)
+			)
+		)
+	)
+	(global_label "SCK"
+		(shape input)
+		(at 127 86.36 0)
+		(fields_autoplaced yes)
+		(effects
+			(font
+				(size 1.27 1.27)
+			)
+			(justify left)
+		)
+		(property "Intersheetrefs" "${INTERSHEET_REFS}"
+			(at 133.7347 86.36 0)
+			(effects
+				(font
